File: kicad/CR2032 Toaster v1.3.sch (KiCad schematic (older format))
At the start: 3 parts, among them J1 Conn_01x01, J2 Conn_01x01

Commit message: Version 1.3
Parts:
- BT1: symbol BAT-HLD-001-THM:BAT-HLD-001-THM -> snapeda:BAT-HLD-001-THM
Changed lines of the file:
@@
 $EndDescr
 $Comp
-L BAT-HLD-001-THM:BAT-HLD-001-THM BT1
+L snapeda:BAT-HLD-001-THM BT1
 U 1 1 60D38724
 P 5550 3450
