File: kicad/CR2032 Toaster_v1.2.kicad_pcb (KiCad board)
At the start: 2 copper layers, 26.5 x 15.5 mm, 6 parts, among them J1 Conn_01x01, J2 Conn_01x01

Commit message: Version 1.3
Parts:
- moved G*** 0.75 mm to (108.0, 110.8)
- moved G*** 0.35 mm to (113.8, 103.0)
Other:
- board text added: "2021/06/27"
- board text added: "JLCJLCJLCJLC"
